Commit message: ackermann engine

File: src/ferrari/urdf/ferrari.xacro (robot description, xacro)
@@ -43,13 +43,59 @@
         </xacro:inertial_box>
     </link>
+    <!-- 앞바퀴용 조향 링크 두 개 추가 -->
+    <link name="front_left_steer_link">
+        <visual>
+            <geometry>
+                <box size="0.01 0.01 0.01"/>
+            </geometry>
+        </visual>
+        <collision>
+            <geometry>
+                <box size="0.01 0.01 0.01"/>
+            </geometry>
+        </collision>
+        <xacro:inertial_box mass="0.02" x="0.01" y="0.01" z="0.01">
+            <origin xyz="0 0 0" rpy="0 0 0"/>
+        </xacro:inertial_box>
+    </link>
+    <link name="front_right_steer_link">
+        <visual>
+            <geometry>
+                <box size="0.01 0.01 0.01"/>
+            </geometry>
+        </visual>
+        <collision>
+            <geometry>
+                <box size="0.01 0.01 0.01"/>
+            </geometry>
+        </collision>
+        <xacro:inertial_box mass="0.02" x="0.01" y="0.01" z="0.01">
+            <origin xyz="0 0 0" rpy="0 0 0"/>
+        </xacro:inertial_box>
+    </link>
+    <!-- 앞바퀴 조향 조인트: yaw 축, ±20deg = ±0.349066rad -->
+    <joint name="front_left_steer_joint" type="revolute">
+        <parent link="base_link"/>
+        <child  link="front_left_steer_link"/>
+        <origin xyz="0.055 0.065 0" rpy="0 0 0"/>   <!-- 원래 앞바퀴 위치와 같게 -->
+        <axis xyz="0 0 1"/>
+        <limit lower="-0.349066" upper="0.349066" effort="30" velocity="2.0"/>
+    </joint>
+    <joint name="front_right_steer_joint" type="revolute">
+        <parent link="base_link"/>
+        <child  link="front_right_steer_link"/>
+        <origin xyz="0.055 -0.065 0" rpy="0 0 0"/>
+        <axis xyz="0 0 1"/>
+        <limit lower="-0.349066" upper="0.349066" effort="30" velocity="2.0"/>
+    </joint>
     <!-- FRONT LEFT WHEEL -->
-    <xacro:wheel_link name="front_left_wheel" parent_link="base_link"
-                  xyz="0.055 0.065 0" rpy="-${pi/2} 0 0" direction="1"/>
+    <xacro:wheel_link name="front_left_wheel" parent_link="front_left_steer_link"
+                  xyz="0 0 0" rpy="-${pi/2} 0 0" direction="1"/>
     <gazebo reference = "front_left_wheel">
         <material>Gazebo/Black</material>
     </gazebo>
     <!-- FRONT RIGHT WHEEL -->
-    <xacro:wheel_link name="front_right_wheel" parent_link="base_link"
-                  xyz="0.055 -0.065 0" rpy="${pi/2} 0 0" direction="-1"/>
+    <xacro:wheel_link name="front_right_wheel" parent_link="front_right_steer_link"
+                  xyz="0 0 0" rpy="${pi/2} 0 0" direction="-1"/>
     <gazebo reference = "front_right_wheel">
         <material>Gazebo/Black</material>
@@ -159,5 +205,6 @@
     </link>
     <!--GAZEBO-->
-    <xacro:include filename="gazebo.xacro"/>
+    <xacro:include filename="ackermann.xacro"/>
+    <xacro:add_gazebo_and_ros2_control/>
     <xacro:include filename="lidar.xacro"/>
     <xacro:include filename="camera.xacro"/>

File: src/ferrari/urdf/macros.xacro (robot description, xacro)
@@ -33,9 +33,10 @@
             <parent link="${parent_link}"/>
             <child link="${name}"/>
-            <origin xyz="${xyz}" rpy="${rpy}"/>
-            <axis xyz="0 0 ${direction}"/>
+            <origin xyz="${xyz}" rpy="0 0 0"/>
+            <axis xyz="0 1 0"/>
         </joint>
         <link name="${name}">
             <visual>
+                <origin xyz="0 0 0" rpy="${rpy}"/>
                 <geometry>
                     <cylinder radius="0.03" length="0.03"/>
@@ -44,4 +45,5 @@
             </visual>
             <collision>
+                <origin xyz="0 0 0" rpy="${rpy}"/>
                 <geometry>
                     <cylinder radius="0.03" length="0.03"/>

Commit message: odometry

File: src/ferrari/urdf/ferrari.xacro (robot description, xacro)
@@ -142,7 +142,7 @@
     <!--LiDAR-->
     <joint name = "laser_joint" type = "fixed">
-        <parent link = "body"/>
+        <parent link = "base_link"/>
         <child link = "laser_frame"/>
-        <origin xyz = "0.1 0 0.075" rpy="0 0 0"/>
+        <origin xyz = "0 0 0.075" rpy="0 0 0"/>
     </joint>
     <link name="laser_frame">
