Commit message: simulator test

File: src/ferrari/urdf/macros.xacro (robot description, xacro)
@@ -40,5 +40,5 @@
                 <origin xyz="0 0 0" rpy="${rpy}"/>
                 <geometry>
-                    <cylinder radius="0.03" length="0.03"/>
+                    <cylinder radius="0.05" length="0.05"/>
                 </geometry>
                 <material name="black"/>
@@ -47,8 +47,8 @@
                 <origin xyz="0 0 0" rpy="${rpy}"/>
                 <geometry>
-                    <cylinder radius="0.03" length="0.03"/>
+                    <cylinder radius="0.05" length="0.05"/>
                 </geometry>
             </collision>
-            <xacro:inertial_cylinder mass="0.1" length="0.03" radius="0.03">
+            <xacro:inertial_cylinder mass="0.1" length="0.05" radius="0.05">
                 <origin xyz="0 0 0" rpy="0 0 0"/>
             </xacro:inertial_cylinder>
