Commit message: rear drive vehicle

File: src/ferrari/urdf/ackermann.xacro (robot description, xacro)
@@ -1,5 +1,4 @@
 <?xml version="1.0"?>
 <robot xmlns:xacro="http://www.ros.org/wiki/xacro">
-  <!-- Gazebo + ros2_control 추가용 매크로 -->
   <xacro:macro name="add_gazebo_and_ros2_control">
     <gazebo>
@@ -12,60 +11,25 @@
         <plugin>gazebo_ros2_control/GazeboSystem</plugin>
       </hardware>
-      <!-- 앞 조향: position -->
+      <!-- 앞 조향: position 제어 -->
       <joint name="front_left_steer_joint">
-        <command_interfaces>
-          <command_interface name="position"/>
-        </command_interfaces>
-        <state_interfaces>
-          <state_interface name="position"/>
-          <state_interface name="velocity"/>
-        </state_interfaces>
+        <command_interface name="position"/>
+        <state_interface   name="position"/>
+        <state_interface   name="velocity"/>
       </joint>
       <joint name="front_right_steer_joint">
-        <command_interfaces>
-          <command_interface name="position"/>
-        </command_interfaces>
-        <state_interfaces>
-          <state_interface name="position"/>
-          <state_interface name="velocity"/>
-        </state_interfaces>
+        <command_interface name="position"/>
+        <state_interface   name="position"/>
+        <state_interface   name="velocity"/>
       </joint>
-      <!-- 앞바퀴 구동이 있다면 여기도 넣고 싶으면 추가 -->
-      <joint name="front_left_wheel_joint">
-        <command_interfaces>
-          <command_interface name="velocity"/>
-        </command_interfaces>
-        <state_interfaces>
-          <state_interface name="position"/>
-          <state_interface name="velocity"/>
-        </state_interfaces>
-      </joint>
-      <joint name="front_right_wheel_joint">
-        <command_interfaces>
-          <command_interface name="velocity"/>
-        </command_interfaces>
-        <state_interfaces>
-          <state_interface name="position"/>
-          <state_interface name="velocity"/>
-        </state_interfaces>
-      </joint>
-      <!-- 뒤 구동: velocity -->
+      <!-- 뒤 구동: velocity 제어 -->
       <joint name="rear_left_wheel_joint">
-        <command_interfaces>
-          <command_interface name="velocity"/>
-        </command_interfaces>
-        <state_interfaces>
-          <state_interface name="position"/>
-          <state_interface name="velocity"/>
-        </state_interfaces>
+        <command_interface name="velocity"/>
+        <state_interface   name="position"/>
+        <state_interface   name="velocity"/>
       </joint>
       <joint name="rear_right_wheel_joint">
-        <command_interfaces>
-          <command_interface name="velocity"/>
-        </command_interfaces>
-        <state_interfaces>
-          <state_interface name="position"/>
-          <state_interface name="velocity"/>
-        </state_interfaces>
+        <command_interface name="velocity"/>
+        <state_interface   name="position"/>
+        <state_interface   name="velocity"/>
       </joint>
     </ros2_control>

Commit message: dual robot setting

File: src/ferrari/urdf/ackermann.xacro (robot description, xacro)
@@ -1,21 +1,32 @@
 <?xml version="1.0"?>
 <robot xmlns:xacro="http://www.ros.org/wiki/xacro">
-  <xacro:macro name="add_gazebo_and_ros2_control">
+  <xacro:macro name="add_gazebo_and_ros2_control" params="joint_suffix:='' controllers_file:='$(find ferrari)/config/controllers.yaml' ros_namespace:='' hardware_name:='ferrari_hw'">
+    <xacro:property name="fl_steer" value="${'front_left_steer_joint' + joint_suffix}"/>
+    <xacro:property name="fr_steer" value="${'front_right_steer_joint' + joint_suffix}"/>
+    <xacro:property name="rl_wheel" value="${'rear_left_wheel_joint' + joint_suffix}"/>
+    <xacro:property name="rr_wheel" value="${'rear_right_wheel_joint' + joint_suffix}"/>
+    <xacro:property name="plugin_name" value="${'gazebo_ros2_control' + joint_suffix}"/>
+    <xacro:property name="hw_name" value="${hardware_name + joint_suffix}"/>
     <gazebo>
-      <plugin name="gazebo_ros2_control" filename="libgazebo_ros2_control.so">
-        <parameters>$(find ferrari)/config/controllers.yaml</parameters>
+      <plugin name="${plugin_name}" filename="libgazebo_ros2_control.so">
+        <xacro:if value="${ros_namespace != ''}">
+          <ros>
+            <namespace>${ros_namespace}</namespace>
+          </ros>
+        </xacro:if>
+        <parameters>${controllers_file}</parameters>
       </plugin>
     </gazebo>
-    <ros2_control name="ferrari_hw" type="system">
+    <ros2_control name="${hw_name}" type="system">
       <hardware>
         <plugin>gazebo_ros2_control/GazeboSystem</plugin>
       </hardware>
       <!-- 앞 조향: position 제어 -->
-      <joint name="front_left_steer_joint">
+      <joint name="${fl_steer}">
         <command_interface name="position"/>
         <state_interface   name="position"/>
         <state_interface   name="velocity"/>
       </joint>
-      <joint name="front_right_steer_joint">
+      <joint name="${fr_steer}">
         <command_interface name="position"/>
         <state_interface   name="position"/>
@@ -23,10 +34,10 @@
       </joint>
       <!-- 뒤 구동: velocity 제어 -->
-      <joint name="rear_left_wheel_joint">
+      <joint name="${rl_wheel}">
         <command_interface name="velocity"/>
         <state_interface   name="position"/>
         <state_interface   name="velocity"/>
       </joint>
-      <joint name="rear_right_wheel_joint">
+      <joint name="${rr_wheel}">
         <command_interface name="velocity"/>
         <state_interface   name="position"/>

File: src/ferrari/urdf/camera.xacro (robot description, xacro)
@@ -1,28 +1,33 @@
 <?xml version="1.0"?>
 <robot xmlns:xacro="http://www.ros.org/wiki/xacro">
-    <gazebo reference="camera_link">
-        <material>Gazebo/Red</material>
-        <sensor name="camera" type="camera">
-            <pose>0 0 0 0 0 0</pose>
-            <visualize>true</visualize>
-            <update_rate>10</update_rate>
-            <camera>
-                <horizontal_fov>1.089</horizontal_fov>
-                <image>
-                    <format>B8G8R8</format>
-                    <width>640</width>
-                    <height>480</height>
-                </image>
-                <clip>
-                    <near>0.05</near>
-                    <far>8.0</far>
-                </clip>
-            </camera>
-            <plugin name="camera_controller" filename="libgazebo_ros_camera.so">
-                <frame_name>camera_link_optical</frame_name>
-                <min_depth>0.1</min_depth>
-                <max_depth>100.0</max_depth>
-            </plugin>
-        </sensor>
-    </gazebo>
+    <xacro:macro name="add_camera" params="frame_suffix:=''">
+        <xacro:property name="camera_link" value="${'camera_link' + frame_suffix}"/>
+        <xacro:property name="camera_optical_link" value="${'camera_link_optical' + frame_suffix}"/>
+        <xacro:property name="camera_sensor_name" value="${'camera' + frame_suffix}"/>
+        <gazebo reference="${camera_link}">
+            <material>Gazebo/Red</material>
+            <sensor name="${camera_sensor_name}" type="camera">
+                <pose>0 0 0 0 0 0</pose>
+                <visualize>true</visualize>
+                <update_rate>10</update_rate>
+                <camera>
+                    <horizontal_fov>1.089</horizontal_fov>
+                    <image>
+                        <format>B8G8R8</format>
+                        <width>640</width>
+                        <height>480</height>
+                    </image>
+                    <clip>
+                        <near>0.05</near>
+                        <far>8.0</far>
+                    </clip>
+                </camera>
+                <plugin name="${'camera_controller' + frame_suffix}" filename="libgazebo_ros_camera.so">
+                    <frame_name>${camera_optical_link}</frame_name>
+                    <min_depth>0.1</min_depth>
+                    <max_depth>100.0</max_depth>
+                </plugin>
+            </sensor>
+        </gazebo>
+    </xacro:macro>
 </robot>

File: src/ferrari/urdf/ferrari.xacro (robot description, xacro)
@@ -1,4 +1,6 @@
 <?xml version="1.0"?>
 <robot xmlns:xacro="http://ros.org/wiki/xacro" name="ferrari" >
+    <xacro:arg name="ros_namespace" default=""/>
+    <xacro:property name="robot_ns" value="$(arg ros_namespace)"/>
     <!--MACROS-->
     <xacro:include filename="macros.xacro"/>
@@ -206,7 +208,10 @@
     <!--GAZEBO-->
     <xacro:include filename="ackermann.xacro"/>
-    <xacro:add_gazebo_and_ros2_control/>
     <xacro:include filename="lidar.xacro"/>
     <xacro:include filename="camera.xacro"/>
     <xacro:include filename="imu.xacro"/>
+    <xacro:add_gazebo_and_ros2_control ros_namespace="${robot_ns}"/>
+    <xacro:add_lidar/>
+    <xacro:add_camera/>
+    <xacro:add_imu/>
 </robot>

File: src/ferrari/urdf/imu.xacro (robot description, xacro)
@@ -1,77 +1,81 @@
 <?xml version="1.0"?>
 <robot xmlns:xacro="http://www.ros.org/wiki/xacro">
-  <!-- imu_link 또는 imu_frame 이름의 링크가 URDF 안에 존재해야 합니다 -->
-  <gazebo reference="imu_link">
-    <material>Gazebo/Blue</material>
-    <!-- Gazebo IMU 센서 정의 -->
-    <sensor name="imu" type="imu">
-      <pose>0 0 0 0 0 0</pose>
-      <visualize>false</visualize>
-      <always_on>true</always_on>
-      <update_rate>100</update_rate>
-      <!-- 노이즈 모델: 가우시안 예시값. 필요에 따라 조정 -->
-      <imu>
-        <angular_velocity>
-          <x>
-            <noise type="gaussian">
-              <mean>0.0</mean>
-              <stddev>0.002</stddev>
-              <bias_mean>0.0</bias_mean>
-              <bias_stddev>0.0002</bias_stddev>
-            </noise>
-          </x>
-          <y>
-            <noise type="gaussian">
-              <mean>0.0</mean>
-              <stddev>0.002</stddev>
-              <bias_mean>0.0</bias_mean>
-              <bias_stddev>0.0002</bias_stddev>
-            </noise>
-          </y>
-          <z>
-            <noise type="gaussian">
-              <mean>0.0</mean>
-              <stddev>0.002</stddev>
-              <bias_mean>0.0</bias_mean>
-              <bias_stddev>0.0002</bias_stddev>
-            </noise>
-          </z>
-        </angular_velocity>
-        <linear_acceleration>
-          <x>
-            <noise type="gaussian">
-              <mean>0.0</mean>
-              <stddev>0.1</stddev>
-              <bias_mean>0.0</bias_mean>
-              <bias_stddev>0.01</bias_stddev>
-            </noise>
-          </x>
-          <y>
-            <noise type="gaussian">
-              <mean>0.0</mean>
-              <stddev>0.1</stddev>
-              <bias_mean>0.0</bias_mean>
-              <bias_stddev>0.01</bias_stddev>
-            </noise>
-          </y>
-          <z>
-            <noise type="gaussian">
-              <mean>0.0</mean>
-              <stddev>0.1</stddev>
-              <bias_mean>0.0</bias_mean>
-              <bias_stddev>0.01</bias_stddev>
-            </noise>
-          </z>
-        </linear_acceleration>
-      </imu>
-      <!-- ROS2 Foxy + Gazebo Classic용 IMU 플러그인 -->
-      <plugin name="imu_plugin" filename="libgazebo_ros_imu_sensor.so">
-        <ros>
-          <!-- ~/out 기본 토픽을 원하는 이름으로 리매핑 -->
-          <argument>~/out:=imu/data</argument>
-        </ros>
-        <frame_name>imu_link</frame_name>
-      </plugin>
-    </sensor>
-  </gazebo>
+  <xacro:macro name="add_imu" params="frame_suffix:=''">
+    <xacro:property name="imu_link_name" value="${'imu_link' + frame_suffix}"/>
+    <xacro:property name="imu_sensor_name" value="${'imu' + frame_suffix}"/>
+    <!-- imu_link 또는 imu_frame 이름의 링크가 URDF 안에 존재해야 합니다 -->
+    <gazebo reference="${imu_link_name}">
+      <material>Gazebo/Blue</material>
+      <!-- Gazebo IMU 센서 정의 -->
+      <sensor name="${imu_sensor_name}" type="imu">
+        <pose>0 0 0 0 0 0</pose>
+        <visualize>false</visualize>
+        <always_on>true</always_on>
+        <update_rate>100</update_rate>
+        <!-- 노이즈 모델: 가우시안 예시값. 필요에 따라 조정 -->
+        <imu>
+          <angular_velocity>
+            <x>
+              <noise type="gaussian">
+                <mean>0.0</mean>
+                <stddev>0.002</stddev>
+                <bias_mean>0.0</bias_mean>
+                <bias_stddev>0.0002</bias_stddev>
+              </noise>
+            </x>
+            <y>
+              <noise type="gaussian">
+                <mean>0.0</mean>
+                <stddev>0.002</stddev>
+                <bias_mean>0.0</bias_mean>
+                <bias_stddev>0.0002</bias_stddev>
+              </noise>
+            </y>
+            <z>
+              <noise type="gaussian">
+                <mean>0.0</mean>
+                <stddev>0.002</stddev>
+                <bias_mean>0.0</bias_mean>
+                <bias_stddev>0.0002</bias_stddev>
+              </noise>
+            </z>
+          </angular_velocity>
+          <linear_acceleration>
+            <x>
+              <noise type="gaussian">
+                <mean>0.0</mean>
+                <stddev>0.1</stddev>
+                <bias_mean>0.0</bias_mean>
+                <bias_stddev>0.01</bias_stddev>
+              </noise>
+            </x>
+            <y>
+              <noise type="gaussian">
+                <mean>0.0</mean>
+                <stddev>0.1</stddev>
+                <bias_mean>0.0</bias_mean>
+                <bias_stddev>0.01</bias_stddev>
+              </noise>
+            </y>
+            <z>
+              <noise type="gaussian">
+                <mean>0.0</mean>
+                <stddev>0.1</stddev>
+                <bias_mean>0.0</bias_mean>
+                <bias_stddev>0.01</bias_stddev>
+              </noise>
+            </z>
+          </linear_acceleration>
+        </imu>
+        <!-- ROS2 Foxy + Gazebo Classic용 IMU 플러그인 -->
+        <plugin name="${'imu_plugin' + frame_suffix}" filename="libgazebo_ros_imu_sensor.so">
+          <ros>
+            <!-- ~/out 기본 토픽을 원하는 이름으로 리매핑 -->
+            <argument>~/out:=imu/data</argument>
+          </ros>
+          <frame_name>${imu_link_name}</frame_name>
+        </plugin>
+      </sensor>
+    </gazebo>
+  </xacro:macro>
 </robot>

File: src/ferrari/urdf/lidar.xacro (robot description, xacro)
@@ -1,31 +1,35 @@
 <?xml version="1.0"?>
 <robot xmlns:xacro="http://www.ros.org/wiki/xacro">
-    <gazebo reference="laser_frame">
-        <material>Gazebo/Red</material>
-        <sensor name="laser" type="ray">
-            <pose>0 0 0 0 0 0</pose>
-            <visualize>true</visualize>
-            <update_rate>10</update_rate>
-            <ray>
-                <scan>
-                    <horizontal>
-                        <samples>360</samples>
-                        <min_angle>-3.14</min_angle>
-                        <max_angle>3.14</max_angle>
-                    </horizontal>
-                </scan>
-                <range>
-                    <min>0.3</min>
-                    <max>12</max>
-                </range>
-            </ray>
-            <plugin name="laser_controller" filename="libgazebo_ros_ray_sensor.so">
-                <ros>
-                    <argument>~/out:=scan</argument>
-                </ros>
-                <output_type>sensor_msgs/LaserScan</output_type>
-                <frame_name>laser_frame</frame_name>
-            </plugin>
-        </sensor>
-    </gazebo>
+    <xacro:macro name="add_lidar" params="frame_suffix:=''">
+        <xacro:property name="lidar_frame" value="${'laser_frame' + frame_suffix}"/>
+        <xacro:property name="lidar_sensor_name" value="${'laser' + frame_suffix}"/>
+        <gazebo reference="${lidar_frame}">
+            <material>Gazebo/Red</material>
+            <sensor name="${lidar_sensor_name}" type="ray">
+                <pose>0 0 0 0 0 0</pose>
+                <visualize>true</visualize>
+                <update_rate>10</update_rate>
+                <ray>
+                    <scan>
+                        <horizontal>
+                            <samples>360</samples>
+                            <min_angle>-3.14</min_angle>
+                            <max_angle>3.14</max_angle>
+                        </horizontal>
+                    </scan>
+                    <range>
+                        <min>0.3</min>
+                        <max>12</max>
+                    </range>
+                </ray>
+                <plugin name="${'laser_controller' + frame_suffix}" filename="libgazebo_ros_ray_sensor.so">
+                    <ros>
+                        <argument>~/out:=scan</argument>
+                    </ros>
+                    <output_type>sensor_msgs/LaserScan</output_type>
+                    <frame_name>${lidar_frame}</frame_name>
+                </plugin>
+            </sensor>
+        </gazebo>
+    </xacro:macro>
 </robot>

File: src/ferrari/urdf/macros.xacro (robot description, xacro)
@@ -29,6 +29,7 @@
     </xacro:macro>
     <!-- wheel macro -->
-    <xacro:macro name="wheel_link" params="name parent_link xyz rpy direction">
-        <joint name="${name}_joint" type="continuous">
+    <xacro:macro name="wheel_link" params="name parent_link xyz rpy direction joint_name:=''">
+        <xacro:property name="wheel_joint_name" value="${joint_name if joint_name else name + '_joint'}"/>
+        <joint name="${wheel_joint_name}" type="continuous">
             <parent link="${parent_link}"/>
             <child link="${name}"/>
