Commit message: sensor topic name update

File: src/ferrari/urdf/camera.xacro (robot description, xacro)
@@ -1,11 +1,12 @@
 <?xml version="1.0"?>
 <robot xmlns:xacro="http://www.ros.org/wiki/xacro">
-    <xacro:macro name="add_camera" params="frame_suffix:=''">
+    <xacro:macro name="add_camera" params="frame_suffix:='' ros_namespace:='' camera_topic_prefix:='camera' camera_sensor_name:='camera'">
         <xacro:property name="camera_link" value="${'camera_link' + frame_suffix}"/>
         <xacro:property name="camera_optical_link" value="${'camera_link_optical' + frame_suffix}"/>
-        <xacro:property name="camera_sensor_name" value="${'camera' + frame_suffix}"/>
+        <xacro:property name="camera_sensor_name_value" value="${camera_sensor_name}"/>
+        <xacro:property name="camera_topic_prefix_full" value="${'/' + ros_namespace + '/' + camera_topic_prefix if ros_namespace != '' else camera_topic_prefix}"/>
         <gazebo reference="${camera_link}">
             <material>Gazebo/Red</material>
-            <sensor name="${camera_sensor_name}" type="camera">
+            <sensor name="${camera_sensor_name_value}" type="camera">
                 <pose>0 0 0 0 0 0</pose>
                 <visualize>true</visualize>
@@ -24,4 +25,8 @@
                 </camera>
                 <plugin name="${'camera_controller' + frame_suffix}" filename="libgazebo_ros_camera.so">
+                    <ros>
+                        <argument>~/image_raw:=${camera_topic_prefix_full}/image_raw</argument>
+                        <argument>~/camera_info:=${camera_topic_prefix_full}/camera_info</argument>
+                    </ros>
                     <frame_name>${camera_optical_link}</frame_name>
                     <min_depth>0.1</min_depth>

File: src/ferrari/urdf/ferrari.xacro (robot description, xacro)
@@ -212,6 +212,6 @@
     <xacro:include filename="imu.xacro"/>
     <xacro:add_gazebo_and_ros2_control ros_namespace="${robot_ns}"/>
-    <xacro:add_lidar/>
-    <xacro:add_camera/>
-    <xacro:add_imu/>
+    <xacro:add_lidar ros_namespace="${robot_ns}"/>
+    <xacro:add_camera ros_namespace="${robot_ns}"/>
+    <xacro:add_imu ros_namespace="${robot_ns}"/>
 </robot>

File: src/ferrari/urdf/ferrari_op.xacro (robot description, xacro)
@@ -239,6 +239,6 @@
     <xacro:include filename="imu.xacro"/>
     <xacro:add_gazebo_and_ros2_control joint_suffix="${suffix}" controllers_file="$(find ferrari)/config/controllers_op.yaml" ros_namespace="${robot_ns}" hardware_name="ferrari_op_hw"/>
-    <xacro:add_lidar frame_suffix="${suffix}"/>
-    <xacro:add_camera frame_suffix="${suffix}"/>
-    <xacro:add_imu frame_suffix="${suffix}"/>
+    <xacro:add_lidar frame_suffix="${suffix}" ros_namespace="${robot_ns}"/>
+    <xacro:add_camera frame_suffix="${suffix}" ros_namespace="${robot_ns}"/>
+    <xacro:add_imu frame_suffix="${suffix}" ros_namespace="${robot_ns}"/>
 </robot>

File: src/ferrari/urdf/imu.xacro (robot description, xacro)
@@ -1,7 +1,8 @@
 <?xml version="1.0"?>
 <robot xmlns:xacro="http://www.ros.org/wiki/xacro">
-  <xacro:macro name="add_imu" params="frame_suffix:=''">
+  <xacro:macro name="add_imu" params="frame_suffix:='' ros_namespace:=''">
     <xacro:property name="imu_link_name" value="${'imu_link' + frame_suffix}"/>
     <xacro:property name="imu_sensor_name" value="${'imu' + frame_suffix}"/>
+    <xacro:property name="imu_topic" value="${'/' + ros_namespace + '/imu/data' if ros_namespace != '' else 'imu/data'}"/>
     <!-- imu_link 또는 imu_frame 이름의 링크가 URDF 안에 존재해야 합니다 -->
     <gazebo reference="${imu_link_name}">
@@ -72,5 +73,5 @@
           <ros>
             <!-- ~/out 기본 토픽을 원하는 이름으로 리매핑 -->
-            <argument>~/out:=imu/data</argument>
+            <argument>~/out:=${imu_topic}</argument>
           </ros>
           <frame_name>${imu_link_name}</frame_name>

File: src/ferrari/urdf/lidar.xacro (robot description, xacro)
@@ -1,7 +1,8 @@
 <?xml version="1.0"?>
 <robot xmlns:xacro="http://www.ros.org/wiki/xacro">
-    <xacro:macro name="add_lidar" params="frame_suffix:=''">
+    <xacro:macro name="add_lidar" params="frame_suffix:='' ros_namespace:=''">
         <xacro:property name="lidar_frame" value="${'laser_frame' + frame_suffix}"/>
         <xacro:property name="lidar_sensor_name" value="${'laser' + frame_suffix}"/>
+        <xacro:property name="lidar_topic" value="${'/' + ros_namespace + '/scan' if ros_namespace != '' else 'scan'}"/>
         <gazebo reference="${lidar_frame}">
             <material>Gazebo/Red</material>
@@ -25,5 +26,5 @@
                 <plugin name="${'laser_controller' + frame_suffix}" filename="libgazebo_ros_ray_sensor.so">
                     <ros>
-                        <argument>~/out:=scan</argument>
+                        <argument>~/out:=${lidar_topic}</argument>
                     </ros>
                     <output_type>sensor_msgs/LaserScan</output_type>
