Commit message: motor success for dual robot

File: src/ferrari/urdf/ferrari_op.xacro (robot description, xacro)
@@ -21,10 +21,11 @@
     <xacro:property name="imu_link_name" value="${'imu_link' + suffix}"/>
     <xacro:property name="body_joint_name" value="${'body_joint' + suffix}"/>
-    <xacro:property name="fl_steer_joint" value="${'front_left_steer_joint' + suffix}"/>
-    <xacro:property name="fr_steer_joint" value="${'front_right_steer_joint' + suffix}"/>
-    <xacro:property name="fl_wheel_joint" value="${'front_left_wheel_joint' + suffix}"/>
-    <xacro:property name="fr_wheel_joint" value="${'front_right_wheel_joint' + suffix}"/>
-    <xacro:property name="rl_wheel_joint" value="${'rear_left_wheel_joint' + suffix}"/>
-    <xacro:property name="rr_wheel_joint" value="${'rear_right_wheel_joint' + suffix}"/>
+    <!-- Actuated joint names는 두 차량이 동일(ros2_control 연동 용) -->
+    <xacro:property name="fl_steer_joint" value="front_left_steer_joint"/>
+    <xacro:property name="fr_steer_joint" value="front_right_steer_joint"/>
+    <xacro:property name="fl_wheel_joint" value="front_left_wheel_joint"/>
+    <xacro:property name="fr_wheel_joint" value="front_right_wheel_joint"/>
+    <xacro:property name="rl_wheel_joint" value="rear_left_wheel_joint"/>
+    <xacro:property name="rr_wheel_joint" value="rear_right_wheel_joint"/>
     <xacro:property name="caster_joint_name" value="${'caster_wheel_joint' + suffix}"/>
     <xacro:property name="laser_joint_name" value="${'laser_joint' + suffix}"/>
@@ -238,5 +239,5 @@
     <xacro:include filename="camera.xacro"/>
     <xacro:include filename="imu.xacro"/>
-    <xacro:add_gazebo_and_ros2_control joint_suffix="${suffix}" controllers_file="$(find ferrari)/config/controllers_op.yaml" ros_namespace="${robot_ns}" hardware_name="ferrari_op_hw"/>
+    <xacro:add_gazebo_and_ros2_control joint_suffix="" controllers_file="$(find ferrari)/config/controllers_op.yaml" ros_namespace="${robot_ns}" hardware_name="ferrari_op_hw"/>
     <xacro:add_lidar frame_suffix="${suffix}" ros_namespace="${robot_ns}"/>
     <xacro:add_camera frame_suffix="${suffix}" ros_namespace="${robot_ns}"/>

Commit message: amcl update

File: src/ferrari/urdf/ferrari_op.xacro (robot description, xacro)
@@ -9,4 +9,5 @@
     <xacro:property name="base_link_name" value="${'base_link' + suffix}"/>
     <xacro:property name="body_link_name" value="${'body' + suffix}"/>
+    <xacro:property name="bar_link_name" value="${'bar' + suffix}"/>
     <xacro:property name="fl_steer_link" value="${'front_left_steer_link' + suffix}"/>
     <xacro:property name="fr_steer_link" value="${'front_right_steer_link' + suffix}"/>
@@ -21,4 +22,5 @@
     <xacro:property name="imu_link_name" value="${'imu_link' + suffix}"/>
     <xacro:property name="body_joint_name" value="${'body_joint' + suffix}"/>
+    <xacro:property name="bar_joint_name" value="${'bar_joint' + suffix}"/>
     <!-- Actuated joint names는 두 차량이 동일(ros2_control 연동 용) -->
     <xacro:property name="fl_steer_joint" value="front_left_steer_joint"/>
@@ -73,4 +75,28 @@
         </xacro:inertial_box>
     </link>
+    <!--BAR LINK-->
+    <joint name = "${bar_joint_name}" type = "fixed">
+        <parent link = "${body_link_name}"/>
+        <child link = "${bar_link_name}" />
+        <origin xyz = "0 0 0.06"/>
+    </joint>
+    <link name = "${bar_link_name}">
+        <visual>
+            <origin xyz = "0 0 0.06"/>
+            <geometry>
+                <box size = "0.05 0.1 0.2"/>
+            </geometry>
+            <material name = "white"/>
+        </visual>
+        <collision>
+            <origin xyz = "0 0 0.06"/>
+            <geometry>
+                <box size = "0.05 0.1 0.2"/>
+            </geometry>
+        </collision>
+        <xacro:inertial_box mass="0.5" x="0.5" y="0.1" z="0.2">
+            <origin xyz="0.0 0 0.06" rpy="0 0 0"/>
+        </xacro:inertial_box>
+    </link>
     <!-- 앞바퀴용 조향 링크 두 개 추가 -->
     <link name="${fl_steer_link}">
